Commit message: HPP : Gripper orientation same as target / Node should be inited by user / Some more utils tool using pinocchio only

File: prl_hpp/urdf_srdf/dummy.urdf (robot description, URDF)
Before this commit: robot dummy, 1 links, 0 joints
Links:
- link base_link: geometry visual box size=0.01 0.025 0.025; visual box size=0.049 0.049 0.049

Commit message: WiP: support as objects

File: prl_hpp/urdf_srdf/dummy.urdf (robot description, URDF)
Before this commit: robot dummy, 1 links, 0 joints
Links:
- removed link base_link
- added link dummy_base; visual box size=0.01 0.025 0.025; visual box size=0.049 0.049 0.049
